File: PCB/Remote_TempHumid/Remote_TempHumid.sch (KiCad schematic (older format))
At the start: 12 parts

Commit message: up to date with old ubuntu
Parts:
- removed C? (x2): 100n, symbol Device:C_Small
- removed C? (x2): 10n, symbol Device:C_Small
- removed U?: ESP-12S, ESP-12S, symbol ESP12S:ESP-12S
- removed U?: STM32F030C8Tx, Package_QFP:LQFP-48_7x7mm_P0.5mm, symbol MCU_ST_STM32F0:STM32F030C8Tx
- added BT1: BK-18650-PC2, 18650_Connector:BAT_BK-18650-PC2, symbol 18650_Holder:BK-18650-PC2
- added C1, C14, C16, C4, C8: 100n, Capacitor_SMD:C_0603_1608Metric, symbol Device:C_Small
- added C15, C17: 4.7u, Capacitor_SMD:C_0603_1608Metric, symbol Device:CP_Small
- added C2, C5, C6, C7: 12p, Capacitor_SMD:C_0603_1608Metric, symbol Device:C_Small
- added D4: D_Schottky, Diode_SMD:D_SMA, symbol Device:D_Schottky
- added D5: LED, LED_SMD:LED_0603_1608Metric, symbol Device:LED_Small_ALT
- added J2: Conn_02x04_Odd_Even, Connector_PinHeader_2.54mm:PinHeader_2x04_P2.54mm_Vertical, symbol Connector_Generic:Conn_02x04_Odd_Even
- added J3: C10418, Custom_lib:C10418, symbol CustomLib:C10418
- added J4: Conn_01x02_Female, Connector_PinSocket_2.54mm:PinSocket_1x02_P2.54mm_Vertical, symbol Connector:Conn_01x02_Female
- added Q1: Q_PMOS_GSD, Package_TO_SOT_SMD:SOT-23W, symbol Device:Q_PMOS_GSD
- added Q2, Q3: Q_NMOS_GSD, Package_TO_SOT_SMD:SOT-23W, symbol Device:Q_NMOS_GSD
- added R10, R11, R12: 10k, Resistor_SMD:R_0603_1608Metric, symbol Device:R_Small
- added R13, R14: 22, Resistor_SMD:R_0603_1608Metric, symbol Device:R_Small
- added R15: 1k, Resistor_SMD:R_0603_1608Metric, symbol Device:R_Small
- added R2: 390, Resistor_SMD:R_0603_1608Metric, symbol Device:R_Small
- added R3, R4: 4.7k, Resistor_SMD:R_0603_1608Metric, symbol Device:R_Small
- added R9: 1.5k, Resistor_SMD:R_0603_1608Metric, symbol Device:R_Small
- added TP3, TP4: TestPoint, TestPoint:TestPoint_Pad_D1.5mm, symbol Connector:TestPoint
- added U1: STM32F103C8Tx, Package_QFP:LQFP-48_7x7mm_P0.5mm, symbol MCU_ST_STM32F1:STM32F103C8Tx
- added U6: ESP-01, ESP8266:ESP-01, symbol ESP8266:ESP-01
- added Y2: 12MHz, Crystal:Crystal_SMD_3225-4Pin_3.2x2.5mm, symbol Device:Crystal_GND24
- C3: renamed from C?; footprint (none) -> Capacitor_SMD:C_0603_1608Metric; LCSC (none) -> C19666
- J1: renamed from J?; footprint (none) -> Connector_PinHeader_2.54mm:PinHeader_1x05_P2.54mm_Vertical
- R1: renamed from R?; footprint (none) -> Resistor_SMD:R_0603_1608Metric; LCSC (none) -> C25804
- U2: renamed from U?; value SHT20 -> SHT21; footprint DFN300X300X110-7N -> SHT20:DFN300X300X110-7N; LCSC C53865 -> C84828
- Y1: renamed from Y?; value Crystal -> 32.768 kHz; footprint (none) -> Crystal:Crystal_SMD_3215-2Pin_3.2x1.5mm; LCSC (none) -> C32346
- gave numbers to parts that had none: 1
Connections:
- net labels added: ESP_EN, ESP_PROG, GPIO2, GPIO4, GPIO5, GPIO6, GPIO7, HSE_0, HSE_1, I2C_SCL, I2C_SDA, LED0, LORA_EN, LSE_0, LSE_1, RX_ESP, SPI_CS, SPI_MISO, SPI_MOSI, SPI_SCK, TX_ESP, UART_RX, UART_TX, USBD+, USBD-, VCC, VCC_STLINK, Vcc_Sensor
- net labels removed: VDD
- wire segments 53 -> 215
- no-connect marks 0 -> 23
Other:
- note added: "Extra GPIOs"
- note added: "HSE"
- note added: "LSE"
- note added: "Oscillators"
- note added: "Temperature and humidity sensor"
- note added: "This circuit choses STlink Vcc \nover battery/USB Vcc when available"
- note removed: "Sensor"
- moved on the sheet: J1, R1, U2, Y1
